File: pcb/USB-serial.sch (KiCad schematic (older format))
At the start: 15 parts, among them J3 USB_B, U201 FT231XS

Commit message: fixing broken symbols
Parts:
- C201, C205: symbol FTDI_FT231XS-U_Breakout-rescue:C -> Device:C
- C202: symbol FTDI_FT231XS-U_Breakout-rescue:CP -> Device:CP
- C203, C204: symbol FTDI_FT231XS-U_Breakout-rescue:C_Small -> Device:C_Small
- C206: symbol antena:C_Small -> Device:C_Small
- D201, D202: symbol antena:LED -> Device:LED
- R201, R202, R203, R204, R205: symbol FTDI_FT231XS-U_Breakout-rescue:R -> Device:R
- U201: symbol FTDI_FT231XS-U_Breakout-rescue:FT231XS -> Interface_USB:FT231XS
Changed lines of the file:
@@
 $EndDescr
 $Comp
-L FTDI_FT231XS-U_Breakout-rescue:C C201
+L Device:C C201
 U 1 1 5784B3B5
 P 3050 2650
@@
 $EndComp
 $Comp
-L FTDI_FT231XS-U_Breakout-rescue:FT231XS U201
+L Interface_USB:FT231XS U201
 U 1 1 5784D541
 P 5450 3350
@@
 $EndComp
 $Comp
-L FTDI_FT231XS-U_Breakout-rescue:R R203
+L Device:R R203
 U 1 1 578639DA
 P 4550 3150
@@
 $EndComp
 $Comp
-L FTDI_FT231XS-U_Breakout-rescue:R R202
+L Device:R R202
 U 1 1 57863B0B
 P 4550 3050
@@
 $EndComp
 $Comp
-L FTDI_FT231XS-U_Breakout-rescue:C_Small C203
+L Device:C_Small C203
 U 1 1 5786579A
 P 3600 3600
@@
 $EndComp
 $Comp
-L FTDI_FT231XS-U_Breakout-rescue:C_Small C204
+L Device:C_Small C204
 U 1 1 57865831
 P 3850 3600
@@
 $EndComp
 $Comp
-L FTDI_FT231XS-U_Breakout-rescue:C C205
+L Device:C C205
 U 1 1 57866269
 P 4450 2500
@@
 $EndComp
 $Comp
-L FTDI_FT231XS-U_Breakout-rescue:CP C202
+L Device:CP C202
 U 1 1 57908B23
 P 3350 2650
@@
 $EndComp
 $Comp
-L FTDI_FT231XS-U_Breakout-rescue:R R201
+L Device:R R201
 U 1 1 57909BE0
 P 4450 2750
@@
 	4300 3350 4750 3350
 $Comp
-L antena:C_Small C206
+L Device:C_Small C206
 U 1 1 5F9F22F3
 P 6400 3150
@@
 	6150 3150 6300 3150
 $Comp
-L antena:LED D201
+L Device:LED D201
 U 1 1 5FA07524
 P 6450 3750
@@
 $EndComp
 $Comp
-L antena:LED D202
+L Device:LED D202
 U 1 1 5FA07A34
 P 6600 3850
@@
 $EndComp
 $Comp
-L FTDI_FT231XS-U_Breakout-rescue:R R204
+L Device:R R204
 U 1 1 5FA0E3BF
 P 6850 3750
@@
 $EndComp
 $Comp
-L FTDI_FT231XS-U_Breakout-rescue:R R205
+L Device:R R205
 U 1 1 5FA0EABB
 P 7000 3850

Commit message: Changing USB connector - rerouting
Parts:
- J3: footprint Connector_USB:USB_B_TE_5787834_Vertical -> Connector_USB:USB_B_OST_USB-B1HSxx_Horizontal
Changed lines of the file:
@@
 F 0 "J3" H 2557 3817 50  0000 C CNN
 F 1 "USB_B" H 2557 3726 50  0000 C CNN
-F 2 "Connector_USB:USB_B_TE_5787834_Vertical" H 2650 3300 50  0001 C CNN
+F 2 "Connector_USB:USB_B_OST_USB-B1HSxx_Horizontal" H 2650 3300 50  0001 C CNN
 F 3 " ~" H 2650 3300 50  0001 C CNN
 	1    2500 3350
