File: pcb/firefly.sch (KiCad schematic (older format))
At the start: 54 parts, among them J101 Conn_02x03_Counter_Clockwise, SW101 SW_DIP_x08, SW102 RESET, U101 ATmega328PB-AU, U102 TLV75733PDBV, U104 AMS1117, Y101 16MHz

Commit message: fixing broken symbols
Parts:
- C101: symbol antena:CP_Small -> Device:CP_Small
- C102, C103, C104, C105, C106, C107, C108, C109, C110, C119, C120, C121, C122, C123, C124: symbol antena:C_Small -> Device:C_Small
- D101, D103, D104, D105: symbol antena:LED -> Device:LED
- D102: symbol antena:D_Schottky_Small -> Device:D_Schottky_Small
- JP109: symbol antena:Jumper -> Device:Jumper
- R1, R101, R102, R103, R104, R106, R2: symbol antena:R -> Device:R
- Y101: symbol antena:Crystal_Small -> Device:Crystal_Small
Changed lines of the file:
@@
 	7600 750  7600 2850
 $Comp
-L antena:LED D101
+L Device:LED D101
 U 1 1 5F686D71
 P 6150 3300
@@
 	6900 3050 6900 2950
 $Comp
-L antena:R R103
+L Device:R R103
 U 1 1 5F6971B6
 P 6550 3300
@@
 $EndComp
 $Comp
-L antena:R R102
+L Device:R R102
 U 1 1 5F725A3C
 P 3200 7100
@@
 	3550 1050 3550 1300
 $Comp
-L antena:R R101
+L Device:R R101
 U 1 1 5F7EA38F
 P 2400 2500
@@
 SW_4
 $Comp
-L antena:Crystal_Small Y101
+L Device:Crystal_Small Y101
 U 1 1 5F9853A3
 P 2300 3350
@@
 $EndComp
 $Comp
-L antena:C_Small C106
+L Device:C_Small C106
 U 1 1 5F986661
 P 2000 3200
@@
 $EndComp
 $Comp
-L antena:C_Small C107
+L Device:C_Small C107
 U 1 1 5F986CA0
 P 2000 3500
@@
 Connection ~ 2300 3200
 $Comp
-L antena:C_Small C108
+L Device:C_Small C108
 U 1 1 5F9AC920
 P 4300 4100
@@
 $EndComp
 $Comp
-L antena:C_Small C102
+L Device:C_Small C102
 U 1 1 5F9BE6D9
 P 900 4250
@@
 $EndComp
 $Comp
-L antena:C_Small C103
+L Device:C_Small C103
 U 1 1 5F9BEAEC
 P 1200 4250
@@
 $EndComp
 $Comp
-L antena:C_Small C104
+L Device:C_Small C104
 U 1 1 5F9D8B6F
 P 1500 4250
@@
 $EndComp
 $Comp
-L antena:C_Small C105
+L Device:C_Small C105
 U 1 1 5F9D8E99
 P 1800 4250
@@
 	900  4350 900  4450
 $Comp
-L antena:CP_Small C101
+L Device:CP_Small C101
 U 1 1 5F9FCC56
 P 900 3500
@@
 	6150 1800 6150 1900
 $Comp
-L antena:D_Schottky_Small D102
+L Device:D_Schottky_Small D102
 U 1 1 5FBEBBBC
 P 6150 1050
@@
 	5650 1050 5650 1400
 $Comp
-L antena:C_Small C109
+L Device:C_Small C109
 U 1 1 5FC0318D
 P 5500 1700
@@
 $EndComp
 $Comp
-L antena:C_Small C110
+L Device:C_Small C110
 U 1 1 5FC03DDE
 P 6600 1700
@@
 $EndComp
 $Comp
-L antena:LED D103
+L Device:LED D103
 U 1 1 5FD38962
 P 6950 1500
@@
 $EndComp
 $Comp
-L antena:R R104
+L Device:R R104
 U 1 1 5FD3931C
 P 6950 1850
@@
 SCK
 $Comp
-L antena:C_Small C119
+L Device:C_Small C119
 U 1 1 5FC8AE3E
 P 900 5050
@@
 $EndComp
 $Comp
-L antena:C_Small C120
+L Device:C_Small C120
 U 1 1 5FC8BC8C
 P 1250 5050
@@
 $EndComp
 $Comp
-L antena:C_Small C121
+L Device:C_Small C121
 U 1 1 5FC8C265
 P 1600 5050
@@
 $EndComp
 $Comp
-L antena:C_Small C122
+L Device:C_Small C122
 U 1 1 5FC8C761
 P 1950 5050
@@
 $EndComp
 $Comp
-L antena:C_Small C123
+L Device:C_Small C123
 U 1 1 5FC8CC1C
 P 2300 5050
@@
 Global decoupling capacitors
 $Comp
-L antena:LED D104
+L Device:LED D104
 U 1 1 5FF42657
 P 5500 4400
@@
 $EndComp
 $Comp
-L antena:LED D105
+L Device:LED D105
 U 1 1 5FF46FF6
 P 5850 4400
@@
 	5500 4150 5500 4250
 $Comp
-L antena:R R1
+L Device:R R1
 U 1 1 5FFD71F9
 P 5500 4800
@@
 $EndComp
 $Comp
-L antena:R R2
+L Device:R R2
 U 1 1 5FFD791C
 P 5850 4800
@@
 	2950 3100 2800 3100
 $Comp
-L antena:R R106
+L Device:R R106
 U 1 1 60248147
 P 2250 2400
@@
 	2250 2500 2200 2500
 $Comp
-L antena:C_Small C124
+L Device:C_Small C124
 U 1 1 60289BFC
 P 2400 2700
@@
 $EndComp
 $Comp
-L antena:Jumper JP109
+L Device:Jumper JP109
 U 1 1 6040C248
 P 6750 700

Commit message: Adding logos, fixing text
Parts:
- removed D101: LED_5V, LED_SMD:LED_0603_1608Metric, symbol Device:LED
- removed JP109: Jumper, Jumper:SolderJumper-2_P1.3mm_Open_RoundedPad1.0x1.5mm, symbol Device:Jumper
- removed R103: 300, Resistor_SMD:R_0603_1608Metric, symbol Device:R
- removed U102: TLV75733PDBV, Package_TO_SOT_SMD:SOT-23-5, symbol Regulator_Linear:TLV75733PDBV
Connections:
- net labels added: +12V
- net labels removed: +5V, 5V
- wire segments 190 -> 180
- no-connect marks 9 -> 7
Other:
- note added: "12V to 5V"
- note removed: "5V to 3.3V"
- moved on the sheet: U104
Changed lines of the file:
@@
 Wire Wire Line
 	7650 1900 8350 1900
-$Comp
-L power:+5V #PWR0101
-U 1 1 5DE4A501
-P 6900 2950
-F 0 "#PWR0101" H 6900 2800 50  0001 C CNN
-F 1 "+5V" H 6915 3123 50  0000 C CNN
-F 2 "" H 6900 2950 50  0001 C CNN
-F 3 "" H 6900 2950 50  0001 C CNN
-	1    6900 2950
-	1    0    0    -1
-$EndComp
 Wire Notes Line
 	5650 6000 5650 7450
@@
 Wire Notes Line
 	7600 750  7600 2850
-$Comp
-L Device:LED D101
-U 1 1 5F686D71
-P 6150 3300
-F 0 "D101" H 6150 3400 50  0000 C CNN
-F 1 "LED_5V" H 6150 3150 50  0000 C CNN
-F 2 "LED_SMD:LED_0603_1608Metric" H 6150 3300 50  0001 C CNN
-F 3 "~" H 6150 3300 50  0001 C CNN
-	1    6150 3300
-	-1   0    0    1
-$EndComp
-Wire Wire Line
-	6900 3050 6900 2950
-$Comp
-L Device:R R103
-U 1 1 5F6971B6
-P 6550 3300
-F 0 "R103" V 6450 3300 50  0000 C CNN
-F 1 "300" V 6550 3300 50  0000 C CNN
-F 2 "Resistor_SMD:R_0603_1608Metric" V 6480 3300 50  0001 C CNN
-F 3 "~" H 6550 3300 50  0001 C CNN
-	1    6550 3300
-	0    1    1    0
-$EndComp
-$Comp
-L power:GND1 #PWR0133
-U 1 1 5F694E04
-P 6800 3300
-F 0 "#PWR0133" H 6800 3050 50  0001 C CNN
-F 1 "GND1" V 6805 3172 50  0000 R CNN
-F 2 "" H 6800 3300 50  0001 C CNN
-F 3 "" H 6800 3300 50  0001 C CNN
-	1    6800 3300
-	0    -1   -1   0
-$EndComp
-Wire Wire Line
-	5500 3050 5900 3050
-Wire Wire Line
-	6800 3300 6700 3300
-Wire Wire Line
-	6400 3300 6300 3300
-Wire Wire Line
-	6000 3300 5900 3300
-Wire Wire Line
-	5900 3300 5900 3050
-Connection ~ 5900 3050
-Wire Wire Line
-	5900 3050 6900 3050
 Wire Notes Line
 	5250 2650 5250 3450
@@
 U 1 1 5F986661
 P 2000 3200
-F 0 "C106" V 1750 3200 50  0000 C CNN
-F 1 "22pF" V 1850 3200 50  0000 C CNN
+F 0 "C106" V 1950 3050 50  0000 C CNN
+F 1 "22pF" V 1950 3350 50  0000 C CNN
 F 2 "Capacitor_SMD:C_0603_1608Metric" H 2000 3200 50  0001 C CNN
 F 3 "~" H 2000 3200 50  0001 C CNN
@@
 Text Label 4550 1050 1    50   ~ 0
 RST
-$Comp
-L Regulator_Linear:TLV75733PDBV U102
-U 1 1 5FB9B859
-P 6150 1500
-F 0 "U102" H 6150 1842 50  0000 C CNN
-F 1 "TLV75733PDBV" H 6150 1751 50  0000 C CNN
-F 2 "Package_TO_SOT_SMD:SOT-23-5" H 6150 1825 50  0001 C CIN
-F 3 "https://www.ti.com/lit/ds/symlink/tlv757p.pdf" H 6150 1550 50  0001 C CNN
-F 4 "https://hr.mouser.com/ProductDetail/Texas-Instruments/TLV75733PDBVR?qs=%2Fha2pyFadugIoPpPm3ZMJDASiJOZ4tX%252BQ8CEtMbd8Pw%2FVXHDUrWd7g%3D%3D" H 6150 1500 50  0001 C CNN "Mouser"
-F 5 "https://lcsc.com/product-detail/Dropout-Regulators-LDO_Texas-Instruments_PTLV75733PDBVR_Texas-Instruments-Texas-Instruments-PTLV75733PDBVR_C189779.html" H 6150 1500 50  0001 C CNN "LCSC"
-	1    6150 1500
-	1    0    0    -1
-$EndComp
 Wire Wire Line
 	5850 1400 5650 1400
-Wire Wire Line
-	5850 1500 5650 1500
-Wire Wire Line
-	5650 1500 5650 1400
 Connection ~ 5650 1400
 Wire Wire Line
@@
 	1    0    0    -1
 $EndComp
-Wire Wire Line
-	6150 1800 6150 1900
 $Comp
 L Device:D_Schottky_Small D102
@@
 	5500 1800 5500 1900
 Text Notes 5250 750  0    118  ~ 0
-5V to 3.3V
+12V to 5V
 Wire Notes Line
 	5250 800  7300 800
@@
 Wire Wire Line
 	2950 2800 2800 2800
-Wire Wire Line
-	2950 2900 2800 2900
-Wire Wire Line
-	2950 3000 2800 3000
 Wire Wire Line
 	2950 3100 2800 3100
@@
 NoConn ~ 2800 2700
 NoConn ~ 2800 2800
-NoConn ~ 2800 2900
-NoConn ~ 2800 3000
 NoConn ~ 2800 3100
 NoConn ~ 4350 2100
@@
 Wire Wire Line
 	2450 2000 2950 2000
-Text Label 6300 4050 2    50   ~ 0
-Vin
-Text Label 7300 4050 0    50   ~ 0
-5V
 Text Label 5500 3050 0    50   ~ 0
-5V
-Wire Wire Line
-	6300 4050 6450 4050
-Wire Wire Line
-	7050 4050 7300 4050
+Vin_fused
 $Comp
 L Regulator_Linear:AMS1117 U104
 U 1 1 6038EE9E
-P 6750 4050
-F 0 "U104" H 6750 4292 50  0000 C CNN
-F 1 "AMS1117" H 6750 4201 50  0000 C CNN
-F 2 "Package_TO_SOT_SMD:SOT-223-3_TabPin2" H 6750 4250 50  0001 C CNN
-F 3 "http://www.advanced-monolithic.com/pdf/ds1117.pdf" H 6850 3800 50  0001 C CNN
-	1    6750 4050
-	1    0    0    -1
-$EndComp
-$Comp
-L power:GND1 #PWR0127
-U 1 1 60390327
-P 6750 4350
-F 0 "#PWR0127" H 6750 4100 50  0001 C CNN
-F 1 "GND1" V 6755 4222 50  0000 R CNN
-F 2 "" H 6750 4350 50  0001 C CNN
-F 3 "" H 6750 4350 50  0001 C CNN
-	1    6750 4350
-	1    0    0    -1
-$EndComp
-$Comp
-L power:+5V #PWR0129
-U 1 1 603A709B
-P 5350 1400
-F 0 "#PWR0129" H 5350 1250 50  0001 C CNN
-F 1 "+5V" H 5365 1573 50  0000 C CNN
-F 2 "" H 5350 1400 50  0001 C CNN
-F 3 "" H 5350 1400 50  0001 C CNN
-	1    5350 1400
-	1    0    0    -1
-$EndComp
-$Comp
-L Device:Jumper JP109
-U 1 1 6040C248
-P 6750 700
-F 0 "JP109" H 6750 964 50  0000 C CNN
-F 1 "Jumper" H 6750 873 50  0000 C CNN
-F 2 "Jumper:SolderJumper-2_P1.3mm_Open_RoundedPad1.0x1.5mm" H 6750 700 50  0001 C CNN
-F 3 "~" H 6750 700 50  0001 C CNN
-	1    6750 700
-	1    0    0    -1
-$EndComp
-$Comp
-L power:+5V #PWR0130
-U 1 1 6040EE4A
-P 6450 700
-F 0 "#PWR0130" H 6450 550 50  0001 C CNN
-F 1 "+5V" H 6465 873 50  0000 C CNN
-F 2 "" H 6450 700 50  0001 C CNN
-F 3 "" H 6450 700 50  0001 C CNN
-	1    6450 700
-	0    -1   -1   0
-$EndComp
-$Comp
-L power:+3.3V #PWR0135
-U 1 1 6040FAE3
-P 7050 700
-F 0 "#PWR0135" H 7050 550 50  0001 C CNN
-F 1 "+3.3V" H 7065 873 50  0000 C CNN
-F 2 "" H 7050 700 50  0001 C CNN
-F 3 "" H 7050 700 50  0001 C CNN
-	1    7050 700
-	0    1    1    0
+P 6150 1400
+F 0 "U104" H 6150 1642 50  0000 C CNN
+F 1 "AMS1117" H 6150 1551 50  0000 C CNN
+F 2 "Package_TO_SOT_SMD:SOT-223-3_TabPin2" H 6150 1600 50  0001 C CNN
+F 3 "http://www.advanced-monolithic.com/pdf/ds1117.pdf" H 6250 1150 50  0001 C CNN
+	1    6150 1400
+	1    0    0    -1
 $EndComp
 $Comp
@@
 	1    0    0    -1
 $EndComp
+Wire Wire Line
+	6150 1700 6150 1900
+Text Label 2050 2900 0    44   ~ 0
+DMX_Enable_Send
+Text Label 2050 3000 0    44   ~ 0
+DMX_Enable_Receive
+Wire Wire Line
+	2050 2900 2950 2900
+Wire Wire Line
+	2050 3000 2950 3000
+$Comp
+L power:+12V #PWR0101
+U 1 1 60660084
+P 5350 1400
+F 0 "#PWR0101" H 5350 1250 50  0001 C CNN
+F 1 "+12V" H 5365 1573 50  0000 C CNN
+F 2 "" H 5350 1400 50  0001 C CNN
+F 3 "" H 5350 1400 50  0001 C CNN
+	1    5350 1400
+	1    0    0    -1
+$EndComp
+$Comp
+L power:+12V #PWR0127
+U 1 1 60661A4B
+P 6600 3050
+F 0 "#PWR0127" H 6600 2900 50  0001 C CNN
+F 1 "+12V" V 6615 3178 50  0000 L CNN
+F 2 "" H 6600 3050 50  0001 C CNN
+F 3 "" H 6600 3050 50  0001 C CNN
+	1    6600 3050
+	0    1    1    0
+$EndComp
+Wire Wire Line
+	5500 3050 6600 3050
 $EndSCHEMATC

Commit message: Adding protection diodes
Parts:
- added D101: 82306120029, Diode_SMD:D_0603_1608Metric, symbol Diode:ESD9B3.3ST5G
- ESD1, ESD2: footprint Diode_SMD:D_SOD-323_HandSoldering -> Diode_SMD:D_SOD-523
- JP3, JP4: footprint Jumper:SolderJumper-2_P1.3mm_Open_RoundedPad1.0x1.5mm -> Jumper:SolderJumper-2_P1.3mm_Bridged_RoundedPad1.0x1.5mm
Connections:
- wire segments 180 -> 181
Other:
- moved on the sheet: TP104
Changed lines of the file:
@@
 F 0 "ESD1" V 10250 6050 50  0000 L CNN
 F 1 "PESD5V0X1UAB" V 10200 5850 50  0000 L CNN
-F 2 "Diode_SMD:D_SOD-323_HandSoldering" H 10100 6150 50  0001 C CNN
+F 2 "Diode_SMD:D_SOD-523" H 10100 6150 50  0001 C CNN
 F 3 "http://www.farnell.com/datasheets/1508358.pdf" H 10100 6150 50  0001 C CNN
 F 4 "PESD5V0X1UAB,115" H 10100 6150 50  0001 C CNN "Article Number"
@@
 Wire Wire Line
 	2850 1600 2850 1300
-Text Label 4250 2000 0    50   ~ 0
-Addressable
 Text Label 2650 1300 0    50   ~ 0
 SW_5
@@
 L Connector:TestPoint_Small TP104
 U 1 1 5FCFE2F0
-P 4250 2000
-F 0 "TP104" H 4150 2100 50  0000 L CNN
-F 1 "TP_A" H 4200 1950 50  0000 L CNN
-F 2 "TestPoint:TestPoint_Pad_D1.0mm" H 4450 2000 50  0001 C CNN
-F 3 "~" H 4450 2000 50  0001 C CNN
-	1    4250 2000
+P 4800 2200
+F 0 "TP104" H 4700 2300 50  0000 L CNN
+F 1 "TP_A" H 4750 2150 50  0000 L CNN
+F 2 "TestPoint:TestPoint_Pad_D1.0mm" H 5000 2200 50  0001 C CNN
+F 3 "~" H 5000 2200 50  0001 C CNN
+	1    4800 2200
 	1    0    0    -1
 $EndComp
@@
 Wire Wire Line
 	2750 1500 2550 1500
-Wire Wire Line
-	4150 2000 4250 2000
 Text Label 2650 3500 0    50   ~ 0
 SCK
@@
 F 0 "ESD2" H 1450 2300 50  0000 L CNN
 F 1 "PESD5V0X1UAB" H 1400 2500 50  0000 L CNN
-F 2 "Diode_SMD:D_SOD-323_HandSoldering" H 1650 2400 50  0001 C CNN
+F 2 "Diode_SMD:D_SOD-523" H 1650 2400 50  0001 C CNN
 F 3 "http://www.farnell.com/datasheets/1508358.pdf" H 1650 2400 50  0001 C CNN
 F 4 "PESD5V0X1UAB,115" H 1650 2400 50  0001 C CNN "Article Number"
@@
 F 0 "JP3" H 8750 5400 50  0000 C CNN
 F 1 "JP_FTDI_TX" H 8700 5600 50  0000 C CNN
-F 2 "Jumper:SolderJumper-2_P1.3mm_Open_RoundedPad1.0x1.5mm" H 8750 5500 50  0001 C CNN
+F 2 "Jumper:SolderJumper-2_P1.3mm_Bridged_RoundedPad1.0x1.5mm" H 8750 5500 50  0001 C CNN
 F 3 "~" H 8750 5500 50  0001 C CNN
 	1    8750 5500
@@
 F 0 "JP4" H 9300 5300 50  0000 C CNN
 F 1 "JP_FTDI_RX" H 9100 5450 50  0000 C CNN
-F 2 "Jumper:SolderJumper-2_P1.3mm_Open_RoundedPad1.0x1.5mm" H 9100 5350 50  0001 C CNN
+F 2 "Jumper:SolderJumper-2_P1.3mm_Bridged_RoundedPad1.0x1.5mm" H 9100 5350 50  0001 C CNN
 F 3 "~" H 9100 5350 50  0001 C CNN
 	1    9100 5350
@@
 Wire Wire Line
 	5500 3050 6600 3050
+$Comp
+L Diode:ESD9B3.3ST5G D101
+U 1 1 607D8D4E
+P 6400 4000
+F 0 "D101" V 6354 4079 50  0000 L CNN
+F 1 "82306120029" H 6300 3900 50  0000 L CNN
+F 2 "Diode_SMD:D_0603_1608Metric" H 6400 4000 50  0001 C CNN
+F 3 "https://hr.mouser.com/datasheet/2/445/82306120029-1724892.pdf" H 6400 4000 50  0001 C CNN
+F 4 "https://hr.mouser.com/ProductDetail/Wurth-Elektronik/82306120029?qs=2kOmHSv6VfRx19zH7vCkmQ%3D%3D" V 6400 4000 50  0001 C CNN "Mouser"
+	1    6400 4000
+	0    1    1    0
+$EndComp
+$Comp
+L power:GND1 #PWR06
+U 1 1 607ECAE5
+P 6400 4200
+F 0 "#PWR06" H 6400 3950 50  0001 C CNN
+F 1 "GND1" V 6405 4072 50  0000 R CNN
+F 2 "" H 6400 4200 50  0001 C CNN
+F 3 "" H 6400 4200 50  0001 C CNN
+	1    6400 4200
+	1    0    0    -1
+$EndComp
+Wire Wire Line
+	6400 3800 6400 3850
+Wire Wire Line
+	6400 4150 6400 4200
+Text Label 6400 3800 1    50   ~ 0
+Vin
 $EndSCHEMATC

Commit message: Adding two connectors with 4 analog inputs
Parts:
- added J102: Analog_1_2, Connector_PinHeader_1.00mm:PinHeader_2x03_P1.00mm_Vertical, symbol Connector_Generic:Conn_02x03_Odd_Even
- added J103: Analog_3_4, Connector_PinHeader_1.00mm:PinHeader_2x03_P1.00mm_Vertical, symbol Connector_Generic:Conn_02x03_Odd_Even
Connections:
- net labels added: A0, A3, A4, A5
- wire segments 181 -> 185
- no-connect marks 7 -> 3
Changed lines of the file:
@@
 NoConn ~ 2750 1900
 NoConn ~ 2750 2100
-NoConn ~ 2800 2600
-NoConn ~ 2800 2700
-NoConn ~ 2800 2800
-NoConn ~ 2800 3100
 NoConn ~ 4350 2100
 Text Label 8300 5350 0    50   ~ 0
@@
 Text Label 6400 3800 1    50   ~ 0
 Vin
+Text Label 2800 2800 0    50   ~ 0
+A3
+Text Label 2800 2700 0    50   ~ 0
+A4
+Text Label 2800 2600 0    50   ~ 0
+A5
+Text Label 2800 3100 0    50   ~ 0
+A0
+$Comp
+L power:+3.3V #PWR0129
+U 1 1 60783E21
+P 6600 4750
+F 0 "#PWR0129" H 6600 4600 50  0001 C CNN
+F 1 "+3.3V" V 6650 4950 50  0000 C CNN
+F 2 "" H 6600 4750 50  0001 C CNN
+F 3 "" H 6600 4750 50  0001 C CNN
+	1    6600 4750
+	0    -1   -1   0
+$EndComp
+$Comp
+L power:+3.3V #PWR0142
+U 1 1 607846E3
+P 7100 4750
+F 0 "#PWR0142" H 7100 4600 50  0001 C CNN
+F 1 "+3.3V" V 7050 5000 50  0000 C CNN
+F 2 "" H 7100 4750 50  0001 C CNN
+F 3 "" H 7100 4750 50  0001 C CNN
+	1    7100 4750
+	0    1    1    0
+$EndComp
+$Comp
+L power:GND1 #PWR0130
+U 1 1 60784E9C
+P 6600 4950
+F 0 "#PWR0130" H 6600 4700 50  0001 C CNN
+F 1 "GND1" V 6700 4950 50  0000 C CNN
+F 2 "" H 6600 4950 50  0001 C CNN
+F 3 "" H 6600 4950 50  0001 C CNN
+	1    6600 4950
+	0    1    1    0
+$EndComp
+$Comp
+L power:GND1 #PWR0143
+U 1 1 607854A8
+P 7100 4950
+F 0 "#PWR0143" H 7100 4700 50  0001 C CNN
+F 1 "GND1" V 7000 4950 50  0000 C CNN
+F 2 "" H 7100 4950 50  0001 C CNN
+F 3 "" H 7100 4950 50  0001 C CNN
+	1    7100 4950
+	0    -1   -1   0
+$EndComp
+Text Label 6500 4850 0    50   ~ 0
+A0
+Text Label 7150 4850 0    50   ~ 0
+A3
+$Comp
+L power:+3.3V #PWR0133
+U 1 1 607B85E6
+P 6600 5350
+F 0 "#PWR0133" H 6600 5200 50  0001 C CNN
+F 1 "+3.3V" V 6650 5550 50  0000 C CNN
+F 2 "" H 6600 5350 50  0001 C CNN
+F 3 "" H 6600 5350 50  0001 C CNN
+	1    6600 5350
+	0    -1   -1   0
+$EndComp
+$Comp
+L power:+3.3V #PWR0144
+U 1 1 607B8CC5
+P 7100 5350
+F 0 "#PWR0144" H 7100 5200 50  0001 C CNN
+F 1 "+3.3V" V 7050 5600 50  0000 C CNN
+F 2 "" H 7100 5350 50  0001 C CNN
+F 3 "" H 7100 5350 50  0001 C CNN
+	1    7100 5350
+	0    1    1    0
+$EndComp
+$Comp
+L power:GND1 #PWR0135
+U 1 1 607B9482
+P 6600 5550
+F 0 "#PWR0135" H 6600 5300 50  0001 C CNN
+F 1 "GND1" V 6700 5550 50  0000 C CNN
+F 2 "" H 6600 5550 50  0001 C CNN
+F 3 "" H 6600 5550 50  0001 C CNN
+	1    6600 5550
+	0    1    1    0
+$EndComp
+$Comp
+L power:GND1 #PWR0145
+U 1 1 607B9B9B
+P 7100 5550
+F 0 "#PWR0145" H 7100 5300 50  0001 C CNN
+F 1 "GND1" V 7000 5550 50  0000 C CNN
+F 2 "" H 7100 5550 50  0001 C CNN
+F 3 "" H 7100 5550 50  0001 C CNN
+	1    7100 5550
+	0    -1   -1   0
+$EndComp
+Wire Wire Line
+	7100 5450 7150 5450
+Wire Wire Line
+	6600 5450 6450 5450
+Text Label 6450 5450 0    50   ~ 0
+A4
+Text Label 7150 5450 0    50   ~ 0
+A5
+$Comp
+L Connector_Generic:Conn_02x03_Odd_Even J102
+U 1 1 607EEFFD
+P 6800 4850
+F 0 "J102" H 6850 5167 50  0000 C CNN
+F 1 "Analog_1_2" H 6850 5076 50  0000 C CNN
+F 2 "Connector_PinHeader_1.00mm:PinHeader_2x03_P1.00mm_Vertical" H 6800 4850 50  0001 C CNN
+F 3 "~" H 6800 4850 50  0001 C CNN
+	1    6800 4850
+	1    0    0    -1
+$EndComp
+$Comp
+L Connector_Generic:Conn_02x03_Odd_Even J103
+U 1 1 607EFEAA
+P 6800 5450
+F 0 "J103" H 6850 5767 50  0000 C CNN
+F 1 "Analog_3_4" H 6850 5676 50  0000 C CNN
+F 2 "Connector_PinHeader_1.00mm:PinHeader_2x03_P1.00mm_Vertical" H 6800 5450 50  0001 C CNN
+F 3 "~" H 6800 5450 50  0001 C CNN
+	1    6800 5450
+	1    0    0    -1
+$EndComp
+Wire Wire Line
+	7100 4850 7150 4850
+Wire Wire Line
+	6600 4850 6500 4850
 $EndSCHEMATC
