File: pcb/firefly.kicad_sch (KiCad schematic)
At the start: 42 parts, among them J101 Conn_02x03_Counter_Clockwise, J102 Analog_1_2, J103 Analog_3_4, SW101 SW_DIP_x08, U1 Pico, U104 AMS1117

Commit message: unesene stavke koje su falile
Other:
- note added: "${project_creator} License: ${project_license} Year: ${project_year}"
- note added: "BOTTOM VIEW"
- note added: "TOP VIEW"
- moved on the sheet: C101, C102, C103, C104, C105, C108, J101, TP104, TP105, U1
